File: Control PCBs/ADC Scaling.sch (EAGLE design)
At the start: 25 parts, among them K1 G5V-2, K2 G5V-2, K3 G5V-2, K4 G5V-2

Commit message: +Flip out connector on scaling pcb to aid in routing the adc +Routed ADC part of ADC/DAC board
Connections:
- net GND: now also JP2.1; no longer JP2.2
- net N$21: now also JP2.2; no longer JP2.1
Changed lines of the file:
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@@
 <segment>
 <pinref part="GND7" gate="1" pin="GND"/>
-<pinref part="JP2" gate="G$1" pin="2"/>
-<wire x1="111.76" y1="40.64" x2="116.84" y2="40.64" width="0.1524" layer="91"/>
-<wire x1="116.84" y1="40.64" x2="119.38" y2="43.18" width="0.1524" layer="91"/>
+<wire x1="111.76" y1="40.64" x2="124.46" y2="40.64" width="0.1524" layer="91"/>
+<wire x1="124.46" y1="40.64" x2="124.46" y2="48.26" width="0.1524" layer="91"/>
+<pinref part="JP2" gate="G$1" pin="1"/>
+<wire x1="124.46" y1="48.26" x2="119.38" y2="48.26" width="0.1524" layer="91"/>
+<wire x1="119.38" y1="48.26" x2="119.38" y2="45.72" width="0.1524" layer="91"/>
 </segment>
 <segment>
@@
 <net name="N$21" class="0">
 <segment>
-<pinref part="JP2" gate="G$1" pin="1"/>
-<wire x1="116.84" y1="45.72" x2="119.38" y2="45.72" width="0.1524" layer="91"/>
 <pinref part="R1" gate="G$1" pin="1"/>
 <wire x1="27.94" y1="55.88" x2="27.94" y2="50.8" width="0.1524" layer="91"/>
@@
 <pinref part="C1" gate="G$1" pin="1"/>
 <junction x="104.14" y="50.8"/>
-</segment>
-</net>
+<pinref part="JP2" gate="G$1" pin="2"/>
+<wire x1="119.38" y1="43.18" x2="116.84" y2="43.18" width="0.1524" layer="91"/>
+<wire x1="116.84" y1="43.18" x2="116.84" y2="45.72" width="0.1524" layer="91"/>
+</segment>
+</net>
